File: hardware/rpi-cm4-carrier-template/cm4-high-speed.kicad_sch (KiCad schematic)
At the start: 1 part

Commit message: Completed PCB Layout
Parts:
- Module1: footprint CM4IO:Raspberry-Pi-4-Compute-Module -> CM4IO:MUnitA
Changed lines of the file:
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@@
     (property "Reference" "Module1" (id 0) (at 73.66 33.02 0))
     (property "Value" "ComputeModule4-CM4" (id 1) (at 73.66 35.56 0))
-    (property "Footprint" "CM4IO:Raspberry-Pi-4-Compute-Module" (id 2) (at 76.2 133.35 0)
+    (property "Footprint" "CM4IO:MUnitA" (id 2) (at 76.2 133.35 0)
       (effects (font (size 1.27 1.27)) hide)
     )
