File: hardware/rpi-cm4-carrier-template/rpi-cm4-carrier-template.kicad_pcb (KiCad board)
At the start: 2 copper layers, 40 x 55 mm, 10 parts, among them J1 USB4110-GF-A_REVB, U1 NLV17SZ07DFT2G

Commit message: Completed PCB Layout
Parts:
- Module1: footprint CM4IO:Raspberry-Pi-4-Compute-Module -> CM4IO:MUnitA
- moved U1 61.7 mm to (167.0, 85.1), turned to 90 degrees
- moved J1 58.2 mm to (171.4, 101.5), turned to 90 degrees
- moved R2 58.0 mm to (170.0, 86.2), turned to -90 degrees
- moved CR1 56.4 mm to (173.5, 111.5)
- moved R1 54.4 mm to (171.0, 90.5), turned to 180 degrees
- moved R3 53.3 mm to (171.0, 92.8), turned to 180 degrees
- moved LED1 52.6 mm to (174.0, 85.8)
- moved R4 50.3 mm to (170.0, 82.2), turned to -90 degrees
- moved LED2 41.2 mm to (174.0, 82.2)
- moved Module1 18.0 mm to (163.5, 100.0)
Connections:
- Module1 pad 21: unconnected-(Module1-Pad21) -> /CM4 GPIO/nLED_Activity
- Module1 pad 95: unconnected-(Module1-Pad95) -> /CM4 GPIO/nPWR_LED
Routing:
- net +5V: track 0.00 -> 40.2 mm
- net +3.3V: track 0.00 -> 34.1 mm
- net /CM4 GPIO/nLED_Activity: track 0.00 -> 22.5 mm, vias 0 -> 2
- net Net-(J1-PadA5): track 0.00 -> 14.5 mm
- net Net-(J1-PadB5): track 0.00 -> 9.28 mm
- net /CM4 GPIO/nPWR_LED: track 0.00 -> 5.93 mm
- net Net-(LED2-Pad1): track 0.00 -> 3.31 mm
- net Net-(LED1-Pad1): track 0.00 -> 3.11 mm
- net Net-(R4-Pad2): track 0.00 -> 2.73 mm
- added copper zone on B.Cu, net GND
- added copper zone on F.Cu, net GND
Other:
- board size 40 x 55 mm -> 21.8 x 55 mm
- board text added: "Nicholas Gregg HomeServer Board V1 2021"
- board text removed: "RPi CM4 Carrier Template"
- board text removed: "Receptacle component options: 1.5mm height: 2x Hirose DF40C-100DS-0.4v OR 3.0mm height: 2x Hirose DF40HC(3.0)-100DS-0.4v"
- board text removed: "Wireless Keepout"
- board text removed: "v01"
